Commit message: Update model to use RGBD camera instead of LiDAR

File: turtlebot3_description/urdf/turtlebot3_burger.urdf (robot description, URDF)
Before this commit: robot turtlebot3_burger, 7 links, 6 joints
Links:
- removed link base_scan
- added link rgbd, mass 0.114; collision cylinder length=0.0315 radius=0.055; visual mesh filename=package://turtlebot3_description/meshes/sensors/lds.stl scale=0.001 0.001 0.001
Joints:
- removed joint scan_joint
- added joint rgbd_joint: type fixed, parent base_link, child rgbd, origin xyz=-0.032 0 0.172 rpy=1.57079632679 3.14159265359 1.57079632679
